File: FLQ01A/FLQ01A.brd (EAGLE design)
At the start: 30.5 x 30.5 mm, 30 parts, among them J1 M10SMD_MALE, J2 M10SMD_MALE, U1 LPC812TSSOP20, U2 EKMBTO5, U3 HTU21DSMD, U4 MMA8452Q, U5 VCNL4000, U6 MPL3115A2LGA8, U7 MMDT3904, Y1 12MHZ

Commit message: [pcb] kick off rev2
Parts:
- added J3: (no value), SparkFun-Connectors:1X04_NO_SILK
- added U$2: (no value), flukso:FLUKSO_LOGO_MEDIUM
- moved U4 1.27 mm to (19.3, 4.57)
- moved C4 1.08 mm to (16.8, 5.84)
- moved C3 0.92 mm to (10.2, 2.54)
- moved C6 0.92 mm to (6.35, 1.78), turned to 270 degrees
- moved C5 0.51 mm to (20.3, 7.37)
- moved U3 0.51 mm to (13.0, 3.05)
- moved R8 0.25 mm to (20.3, 8.64)
Connections:
- net 3.3V: now also J3.4
- net GND: now also J3.1
- net I2C0_SCL: now also J3.3
- net I2C0_SDA: now also J3.2
Routing:
- net 3.3V: track 90.3 -> 103.6 mm
- net I2C0_SCL: track 45.4 -> 57.6 mm, vias 3 -> 4
- net I2C0_SDA: track 46.8 -> 55.2 mm
- net GND: vias 14 -> 15
Other:
- board text added: "13/01/14"
- board text added: "GND"
- board text added: "SCL"
- board text added: "SDA"
- board text added: "VCC"
- board text added: "r2"
- board text removed: "03/01/14"
- board text removed: "r1"
