File: FLQ01A/FLQ01A.sch (EAGLE design)
At the start: 30 parts, among them J1 M10SMD_MALE, J2 M10SMD_MALE, U1 LPC812TSSOP20, U2 EKMBTO5, U3 HTU21DSMD, U4 MMA8452Q, U5 VCNL4000, U6 MPL3115A2LGA8, U7 MMDT3904, Y1 12MHZ

Commit message: [pcb] kick off rev2
Parts:
- added J3: (no value), SparkFun-Connectors:M041X04_NO_SILK
Connections:
- net 3.3V: now also J3.4
- net GND: now also J3.1
- net I2C0_SCL: now also J3.3
- net I2C0_SDA: now also J3.2
Other:
- note added: "2"
- note removed: "1"
Changed lines of the file:
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@@
 <part name="R9" library="SparkFun-Passives" deviceset="RESISTOR" device="0402-RES" value="10k"/>
 <part name="GND17" library="SparkFun-Aesthetics" deviceset="GND" device=""/>
+<part name="J3" library="SparkFun-Connectors" deviceset="M04" device="1X04_NO_SILK"/>
+<part name="GND18" library="SparkFun-Aesthetics" deviceset="GND" device=""/>
+<part name="SUPPLY9" library="SparkFun-Aesthetics" deviceset="3.3V" device=""/>
 </parts>
 <sheets>
 <sheet>
 <plain>
-<text x="256.54" y="7.62" size="2.54" layer="91">1</text>
+<text x="256.54" y="7.62" size="2.54" layer="91">2</text>
 <text x="165.1" y="33.02" size="1.778" layer="91">Copyright (c) 2014 Flukso</text>
 <text x="165.1" y="30.48" size="1.778" layer="91">Licensed under CERN OHL v1.2</text>
@@
 <instance part="R9" gate="G$1" x="248.92" y="137.16" rot="R90"/>
 <instance part="GND17" gate="1" x="248.92" y="111.76"/>
+<instance part="J3" gate="G$1" x="17.78" y="119.38"/>
+<instance part="GND18" gate="1" x="25.4" y="114.3"/>
+<instance part="SUPPLY9" gate="G$1" x="25.4" y="124.46"/>
 </instances>
 <busses>
@@
 <wire x1="248.92" y1="121.92" x2="248.92" y2="114.3" width="0.1524" layer="91"/>
 </segment>
+<segment>
+<pinref part="J3" gate="G$1" pin="1"/>
+<wire x1="22.86" y1="116.84" x2="25.4" y2="116.84" width="0.1524" layer="91"/>
+<pinref part="GND18" gate="1" pin="GND"/>
+</segment>
 </net>
 <net name="PIO0_17" class="0">
@@
 <label x="132.08" y="27.94" size="1.27" layer="95" xref="yes"/>
 </segment>
+<segment>
+<pinref part="J3" gate="G$1" pin="2"/>
+<wire x1="22.86" y1="119.38" x2="25.4" y2="119.38" width="0.1524" layer="91"/>
+<label x="25.4" y="119.38" size="1.27" layer="95" xref="yes"/>
+</segment>
 </net>
 <net name="I2C0_SCL" class="0">
@@
 <wire x1="129.54" y1="30.48" x2="132.08" y2="30.48" width="0.1524" layer="91"/>
 <label x="132.08" y="30.48" size="1.27" layer="95" xref="yes"/>
+</segment>
+<segment>
+<pinref part="J3" gate="G$1" pin="3"/>
+<wire x1="22.86" y1="121.92" x2="25.4" y2="121.92" width="0.1524" layer="91"/>
+<label x="25.4" y="121.92" size="1.27" layer="95" xref="yes"/>
 </segment>
 </net>
@@
 <wire x1="86.36" y1="30.48" x2="86.36" y2="25.4" width="0.1524" layer="91"/>
 </segment>
-</net>
+<segment>
+<pinref part="J3" gate="G$1" pin="4"/>
+<wire x1="22.86" y1="124.46" x2="25.4" y2="124.46" width="0.1524" layer="91"/>
+<pinref part="SUPPLY9" gate="G$1" pin="3.3V"/>
+</segment>
+</net>
