File: FLT04A/FLT04A.brd (EAGLE design)
At the start: 30.5 x 30.5 mm, 26 parts, among them J1 M10", J2 M10", U1 741G04, U4 3.3V/150mA

Commit message: [flt] add pull-up to ISP_EN pin
Parts:
- added R10: 100k, SparkFun-Passives:0402-RES
- moved C2 1.02 mm to (24.1, 9.14)
- moved R3 1.02 mm to (21.1, 7.11)
Connections:
- net !ISP_EN!: now also R10.1
- net 3.3V: now also R10.2
Routing:
- net 3.3V: track 52.4 -> 55.8 mm
- net N$1: track 7.34 -> 6.33 mm
- net !ISP_EN!: track 29.8 -> 30.8 mm
Other:
- board text added: "15/11/14"
- board text added: "FLT04Ar2"
- board text removed: "03/01/14"
- board text removed: "FLT04Ar1"
Changed lines of the file:
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@@
 <wire x1="30.48" y1="30.48" x2="0" y2="30.48" width="0" layer="20"/>
 <wire x1="0" y1="30.48" x2="0" y2="0" width="0" layer="20"/>
-<text x="21.336" y="20.828" size="1.27" layer="21" font="vector" ratio="15" rot="R180">FLT04Ar1</text>
-<text x="29.972" y="23.876" size="0.6096" layer="21" font="vector" ratio="15" rot="R90">03/01/14</text>
+<text x="21.336" y="20.828" size="1.27" layer="21" font="vector" ratio="15" rot="R180">FLT04Ar2</text>
+<text x="29.972" y="23.876" size="0.6096" layer="21" font="vector" ratio="15" rot="R90">15/11/14</text>
 <text x="7.112" y="3.048" size="1.27" layer="21" font="vector" ratio="10" rot="R90">GND</text>
 <text x="22.352" y="3.048" size="1.27" layer="21" font="vector" ratio="10" rot="R90">GND</text>
@@
 <attribute name="NAME" x="15.875" y="9.2075" size="0.4064" layer="25" rot="R180"/>
 </element>
-<element name="R3" library="SparkFun-Passives" package="0402-RES" value="220" x="21.082" y="8.128" smashed="yes" rot="R180">
-<attribute name="NAME" x="20.955" y="9.2075" size="0.4064" layer="25" rot="R180"/>
+<element name="R3" library="SparkFun-Passives" package="0402-RES" value="220" x="21.082" y="7.112" smashed="yes" rot="R180">
+<attribute name="NAME" x="20.955" y="6.4135" size="0.4064" layer="25" rot="R180"/>
 </element>
 <element name="J1" library="SparkFun-Connectors" package="1X10" value="M10&quot;" x="3.81" y="26.67" smashed="yes" rot="R270">
@@
 <attribute name="NAME" x="21.209" y="22.2885" size="0.4064" layer="25"/>
 </element>
-<element name="C2" library="SparkFun-Passives" package="0402-CAP" value="100nF" x="24.13" y="8.128" smashed="yes">
-<attribute name="NAME" x="23.749" y="9.2075" size="0.4064" layer="25" rot="R180"/>
+<element name="C2" library="SparkFun-Passives" package="0402-CAP" value="100nF" x="24.13" y="9.144" smashed="yes">
+<attribute name="NAME" x="25.019" y="10.2235" size="0.4064" layer="25" rot="R180"/>
 </element>
 <element name="U4" library="SparkFun-PowerIC" package="SOT23-5" value="3.3V/150mA" x="9.398" y="5.334" smashed="yes">
@@
 <element name="SJ4" library="SparkFun-Passives" package="SJ_2S" value="SOLDERJUMPERNC" x="9.144" y="8.636" smashed="yes" rot="R90">
 <attribute name="NAME" x="10.4802" y="9.144" size="0.4064" layer="25"/>
+</element>
+<element name="R10" library="SparkFun-Passives" package="0402-RES" value="100k" x="21.082" y="8.382" smashed="yes">
+<attribute name="NAME" x="21.463" y="9.4615" size="0.4064" layer="25" rot="R180"/>
 </element>
 </elements>
@@
 <wire x1="21.59" y1="10.48" x2="21.59" y2="9.906" width="0.254" layer="1"/>
 <wire x1="21.59" y1="9.906" x2="20.432" y2="8.748" width="0.254" layer="1"/>
-<wire x1="20.432" y1="8.748" x2="20.432" y2="8.128" width="0.254" layer="1"/>
+<contactref element="R10" pad="1"/>
+<wire x1="20.432" y1="8.748" x2="20.432" y2="8.382" width="0.254" layer="1"/>
+<wire x1="20.432" y1="8.382" x2="20.432" y2="7.112" width="0.254" layer="1"/>
 </signal>
 <signal name="N$1">
 <contactref element="J3" pad="8"/>
 <contactref element="R3" pad="1"/>
-<wire x1="21.732" y1="8.128" x2="21.732" y2="4.176" width="0.254" layer="1"/>
+<wire x1="21.732" y1="7.112" x2="21.732" y2="4.176" width="0.254" layer="1"/>
 <wire x1="21.732" y1="4.176" x2="24.13" y2="1.778" width="0.254" layer="1"/>
 </signal>
@@
 <wire x1="24.384" y1="16.256" x2="26.67" y2="13.97" width="0.4064" layer="1"/>
 <contactref element="C2" pad="2"/>
-<wire x1="24.78" y1="8.128" x2="24.78" y2="11.796" width="0.254" layer="1"/>
 <wire x1="24.78" y1="11.796" x2="22.606" y2="13.97" width="0.254" layer="1"/>
 <wire x1="22.606" y1="13.97" x2="22.606" y2="14.478" width="0.254" layer="1"/>
@@
 <wire x1="12.192" y1="11.43" x2="12.558" y2="11.796" width="0.4064" layer="1"/>
 <wire x1="12.558" y1="11.796" x2="12.558" y2="12.38" width="0.4064" layer="1"/>
+<contactref element="R10" pad="2"/>
+<wire x1="21.732" y1="8.382" x2="21.732" y2="8.524" width="0.254" layer="1"/>
+<wire x1="24.78" y1="11.796" x2="24.78" y2="9.144" width="0.254" layer="1"/>
+<wire x1="21.732" y1="8.524" x2="22.21" y2="8.524" width="0.254" layer="1"/>
+<wire x1="22.21" y1="8.524" x2="22.86" y2="7.874" width="0.254" layer="1"/>
+<wire x1="22.86" y1="7.874" x2="24.384" y2="7.874" width="0.254" layer="1"/>
+<wire x1="24.384" y1="7.874" x2="24.78" y2="8.27" width="0.254" layer="1"/>
+<wire x1="24.78" y1="8.27" x2="24.78" y2="9.144" width="0.254" layer="1"/>
 </signal>
 <signal name="PIO0_14">

Commit message: [flt] 10uF cap did not connect to GND
Connections:
- removed net N$14: C3.C
- net GND: now also C3.C
Changed lines of the file:
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@@
 <via x="8.382" y="15.748" extent="1-16" drill="0.4064" diameter="0.6096"/>
 <contactref element="U4" pad="2"/>
+<contactref element="C3" pad="C"/>
 </signal>
 <signal name="!RESET!">
@@
 <wire x1="21.448" y1="28.814" x2="21.59" y2="28.702" width="0.254" layer="1"/>
 </signal>
-<signal name="N$14">
-<contactref element="C3" pad="C"/>
-</signal>
 <signal name="N$15">
