File: FLT04A/FLT04A.sch (EAGLE design)
At the start: 26 parts, among them J1 M10", J2 M10", U1 741G04, U4 3.3V/150mA

Commit message: [flt] add pull-up to ISP_EN pin
Parts:
- added R10: 100k, SparkFun-Passives:RESISTOR0402-RES
Connections:
- net !ISP_EN!: now also R10.1
- net 3.3V: now also R10.2
Changed lines of the file:
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@@
 <part name="SJ4" library="SparkFun-Passives" deviceset="SOLDERJUMPER" device="NC"/>
 <part name="SUPPLY5" library="SparkFun-Aesthetics" deviceset="3.3V" device=""/>
+<part name="R10" library="SparkFun-Passives" deviceset="RESISTOR" device="0402-RES" value="100k"/>
 </parts>
 <sheets>
@@
 </instance>
 <instance part="SUPPLY5" gate="G$1" x="223.52" y="96.52"/>
+<instance part="R10" gate="G$1" x="35.56" y="96.52" smashed="yes" rot="R90">
+<attribute name="NAME" x="34.0614" y="92.71" size="1.778" layer="95" rot="R90"/>
+<attribute name="VALUE" x="38.862" y="92.71" size="1.778" layer="96" rot="R90"/>
+</instance>
 </instances>
 <busses>
@@
 <wire x1="58.42" y1="104.14" x2="58.42" y2="101.6" width="0.1524" layer="91"/>
 <junction x="58.42" y="104.14"/>
+<pinref part="R10" gate="G$1" pin="2"/>
+<wire x1="48.26" y1="104.14" x2="35.56" y2="104.14" width="0.1524" layer="91"/>
+<wire x1="35.56" y1="104.14" x2="35.56" y2="101.6" width="0.1524" layer="91"/>
+<junction x="48.26" y="104.14"/>
 </segment>
 <segment>
@@
 </segment>
 <segment>
-<wire x1="48.26" y1="86.36" x2="45.72" y2="86.36" width="0.1524" layer="91"/>
-<label x="45.72" y="86.36" size="1.27" layer="95" font="vector" rot="R180" xref="yes"/>
+<wire x1="48.26" y1="86.36" x2="35.56" y2="86.36" width="0.1524" layer="91"/>
+<label x="35.56" y="86.36" size="1.27" layer="95" font="vector" rot="R180" xref="yes"/>
 <pinref part="U1" gate="G$1" pin="I"/>
-</segment>
-</net>
+<pinref part="R10" gate="G$1" pin="1"/>
+<wire x1="35.56" y1="91.44" x2="35.56" y2="86.36" width="0.1524" layer="91"/>
+</segment>
+</net>

Commit message: [flt] 10uF cap did not connect to GND
Connections:
- removed net N$14: C3.-
- net GND: now also C3.-
Changed lines of the file:
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@@
 <pinref part="GND9" gate="1" pin="GND"/>
+</segment>
+<segment>
+<pinref part="C3" gate="G$1" pin="-"/>
+<pinref part="GND10" gate="1" pin="GND"/>
+<wire x1="208.28" y1="83.82" x2="208.28" y2="81.28" width="0.1524" layer="91"/>
 </segment>
 </net>
@@
 </segment>
 </net>
-<net name="N$14" class="0">
-<segment>
-<pinref part="C3" gate="G$1" pin="-"/>
-<wire x1="208.28" y1="83.82" x2="208.28" y2="81.28" width="0.1524" layer="91"/>
-<pinref part="GND10" gate="1" pin="GND"/>
-</segment>
-</net>
