File: FLK01B/FLK01B.brd (EAGLE design)
At the start: 66 x 30.5 mm, 38 parts, among them J1 M10SMD_MALE_SHORT, J2 M10SMD_MALE_SHORT, J3 M10SMD_FEMALE_SHORT, J4 M10SMD_FEMALE_SHORT, U1 LPC812TSSOP20, U2 EKMBTO5, U3 HTU21DSMD, U4 MMA8452Q, U5 VCNL4010, U6 MPL3115A2LGA8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

Commit message: [flk/r] minor changes to layout
Parts:
- moved C11 0.63 mm to (47.1, 5.71)
- moved U$3 0.63 mm to (50.8, 15.9)
- moved U$7 0.25 mm to (57.4, 27.9)
Connections:
- removed net GND2: J4.6
- removed net RFM_SDI: J2.2, U1.12
- new net MMA_INT: J2.2, U1.12, U4.11
- net AGND: now also J4.6
- net ISP_TXD: no longer U4.11
- net PIO0_1: no longer U$3.SDI
- net PIO0_4: now also U$3.SDI
Routing:
- net MMA_INT: track 0.00 -> 48.8 mm, vias 0 -> 2
- net ISP_TXD: track 41.0 -> 10.7 mm, vias 2 -> 0
- net RFM_SDI: track 22.2 -> 0.00 mm
- net PIO0_4: track 0.00 -> 21.5 mm
- net PIO0_1: track 17.7 -> 0.00 mm, vias 2 -> 0
- net VCC: track 35.5 -> 34.3 mm
- net PIO0_7: track 22.8 -> 21.7 mm
- net N$1: track 6.85 -> 7.49 mm
- net PIO0_13: track 4.99 -> 4.46 mm
