File: FLK01B/FLK01B.sch (EAGLE design)
At the start: 36 parts, among them J1 M10SMD_MALE_SHORT, J2 M10SMD_MALE_SHORT, J3 M10SMD_FEMALE_SHORT, J4 M10SMD_FEMALE_SHORT, U1 LPC812TSSOP20, U2 EKMBTO5, U3 HTU21DSMD, U4 MMA8452Q, U5 VCNL4010, U6 MPL3115A2LGA8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

Commit message: [flk/r] minor changes to layout
Connections:
- removed net GND2: J4.6
- removed net RFM_SDI: J2.2, U1.PIO0_1/ACMP_I2/CLKIN/TDI
- new net MMA_INT: J2.2, U1.PIO0_1/ACMP_I2/CLKIN/TDI, U4.INT1
- net AGND: now also J4.6
- net ISP_TXD: no longer U4.INT1
- net PIO0_1: no longer U$3.SDI
- net PIO0_4: now also U$3.SDI
Other:
- note added: "+RFM_SDI"
Changed lines of the file:
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@@
 <text x="165.1" y="27.94" size="1.778" layer="91">http://ohwr.org/cernohl</text>
 <text x="165.1" y="25.4" size="1.778" layer="91">by bart@flukso.net</text>
+<text x="35.56" y="152.4" size="1.27" layer="91">+RFM_SDI</text>
 </plain>
 <instances>
@@
 <pinref part="J1" gate="G$1" pin="5"/>
 </segment>
-<segment>
-<pinref part="U4" gate="G$1" pin="INT1"/>
-<wire x1="213.36" y1="50.8" x2="218.44" y2="50.8" width="0.1524" layer="91"/>
-<label x="218.44" y="50.8" size="1.27" layer="95" xref="yes"/>
-</segment>
 </net>
 <net name="SWCLK" class="0">
@@
 <segment>
 <pinref part="U4" gate="G$1" pin="SDA"/>
-<wire x1="213.36" y1="58.42" x2="218.44" y2="58.42" width="0.1524" layer="91"/>
-<label x="218.44" y="58.42" size="1.27" layer="95" xref="yes"/>
+<wire x1="213.36" y1="58.42" x2="215.9" y2="58.42" width="0.1524" layer="91"/>
+<label x="215.9" y="58.42" size="1.27" layer="95" xref="yes"/>
 </segment>
 <segment>
@@
 <segment>
 <pinref part="U4" gate="G$1" pin="SCL"/>
-<wire x1="213.36" y1="60.96" x2="218.44" y2="60.96" width="0.1524" layer="91"/>
-<label x="218.44" y="60.96" size="1.27" layer="95" xref="yes"/>
+<wire x1="213.36" y1="60.96" x2="215.9" y2="60.96" width="0.1524" layer="91"/>
+<label x="215.9" y="60.96" size="1.27" layer="95" xref="yes"/>
 </segment>
 <segment>
@@
 <label x="25.4" y="111.76" size="1.27" layer="95" xref="yes"/>
 <pinref part="J2" gate="G$1" pin="3"/>
-</segment>
-</net>
-<net name="RFM_SDI" class="0">
-<segment>
-<pinref part="U1" gate="A" pin="PIO0_1/ACMP_I2/CLKIN/TDI"/>
-<wire x1="223.52" y1="132.08" x2="226.06" y2="132.08" width="0.1524" layer="91"/>
-<label x="226.06" y="132.08" size="1.27" layer="95" xref="yes"/>
-</segment>
-<segment>
-<wire x1="22.86" y1="109.22" x2="25.4" y2="109.22" width="0.1524" layer="91"/>
-<label x="25.4" y="109.22" size="1.27" layer="95" xref="yes"/>
-<pinref part="J2" gate="G$1" pin="2"/>
 </segment>
 </net>
@@
 <pinref part="J3" gate="G$1" pin="5"/>
 </segment>
+<segment>
+<pinref part="U$3" gate="G$1" pin="SDI"/>
+<wire x1="160.02" y1="96.52" x2="157.48" y2="96.52" width="0.1524" layer="91"/>
+<label x="157.48" y="96.52" size="1.27" layer="95" rot="R180" xref="yes"/>
+</segment>
 </net>
 <net name="PIO0_5" class="0">
@@
 <label x="66.04" y="109.22" size="1.27" layer="95" xref="yes"/>
 <pinref part="J4" gate="G$1" pin="2"/>
-</segment>
-<segment>
-<wire x1="160.02" y1="96.52" x2="157.48" y2="96.52" width="0.1524" layer="91"/>
-<label x="157.48" y="96.52" size="1.27" layer="95" rot="R180" xref="yes"/>
-<pinref part="U$3" gate="G$1" pin="SDI"/>
 </segment>
 </net>
@@
 <pinref part="C11" gate="G$1" pin="1"/>
 <wire x1="172.72" y1="109.22" x2="198.12" y2="109.22" width="0.1524" layer="91"/>
+<junction x="172.72" y="109.22"/>
 </segment>
 <segment>
@@
 <wire x1="81.28" y1="86.36" x2="81.28" y2="88.9" width="0.1524" layer="91"/>
 <pinref part="SUPPLY13" gate="G$1" pin="VCC"/>
-</segment>
-</net>
-<net name="GND2" class="0">
-<segment>
-<pinref part="J4" gate="G$1" pin="6"/>
-<wire x1="63.5" y1="119.38" x2="66.04" y2="119.38" width="0.1524" layer="91"/>
-<label x="66.04" y="119.38" size="1.27" layer="95" xref="yes"/>
+<junction x="66.04" y="86.36"/>
 </segment>
 </net>
@@
 <pinref part="U$6" gate="G$1" pin="AGND"/>
 </segment>
-</net>
+<segment>
+<pinref part="J4" gate="G$1" pin="6"/>
+<wire x1="63.5" y1="119.38" x2="66.04" y2="119.38" width="0.1524" layer="91"/>
+<label x="66.04" y="119.38" size="1.27" layer="95" xref="yes"/>
+</segment>
+</net>
+<net name="MMA_INT" class="0">
+<segment>
+<pinref part="U1" gate="A" pin="PIO0_1/ACMP_I2/CLKIN/TDI"/>
+<wire x1="223.52" y1="132.08" x2="226.06" y2="132.08" width="0.1524" layer="91"/>
+<label x="226.06" y="132.08" size="1.27" layer="95" xref="yes"/>
+</segment>
+<segment>
+<pinref part="U4" gate="G$1" pin="INT1"/>
+<wire x1="213.36" y1="50.8" x2="215.9" y2="50.8" width="0.1524" layer="91"/>
+<label x="215.9" y="50.8" size="1.27" layer="95" xref="yes"/>
+</segment>
+<segment>
+<pinref part="J2" gate="G$1" pin="2"/>
+<wire x1="22.86" y1="109.22" x2="25.4" y2="109.22" width="0.1524" layer="91"/>
+<label x="25.4" y="109.22" size="1.27" layer="95" xref="yes"/>
+</segment>
+</net>
